File: Ki_Nema23_TB6600_Arduino_Simple_Accel_7segment/test_Arduino.sch (KiCad schematic (older format))
At the start: 16 parts, among them P1 Power, P2 Analog, P3 Digital, P4 Digital, P5 CONN_01X01, P6 CONN_01X01, P7 CONN_01X01, P8 CONN_01X01

Commit message: 回路図修正
Other:
- note added: "The direction of motor rotation can be reversed by \nreversing the DIR to +/-. Convenient \nwhen you don't want to loosen it because it consists of a right-hand thread."
Changed lines of the file:
@@
 Text Notes 7250 1950 0    50   ~ 0
 red : A+\ngreen : A-\nyellow : B+\nblue : B-
+Text Notes 5950 1000 0    31   ~ 0
+The direction of motor rotation can be reversed by \nreversing the DIR to +/-. Convenient \nwhen you don't want to loosen it because it consists of a right-hand thread.
 $EndSCHEMATC
